File: DummyLoad.brd (EAGLE design)
At the start: 100 x 85.1 mm, 41 parts, among them IC1 LM324N, IC2 PIC18F2550_28DIP, IC3 MAX7219CNG, Q1 MTP3055, SW1 EC11B-V-T, X1 MINI-USB_B, X2 LOAD

Commit message: Update to latest local version
Parts:
- added C9: (no value), rcl:D/7343-31R
- added R21: 10k, rcl:R1206
- moved JP2 3.81 mm to (57.1, 77.9)
- moved R4 2.54 mm to (50.8, 70.0)
- moved Q2 0.95 mm to (73.7, 51.8)
- moved C4 0.63 mm to (71.1, 45.1)
- moved C5 0.63 mm to (76.2, 45.1)
- moved C6 0.63 mm to (67.3, 45.1)
- moved R15 0.63 mm to (59.7, 45.1)
- moved R16 0.63 mm to (81.3, 45.1)
- moved R17 0.63 mm to (85.1, 45.1)
Connections:
- new net N$13: IC3.18, R21.2
- net +5V: now also C9.+, R21.1
- net GND: now also C9.-
Routing:
- net GND: track 192.1 -> 181.1 mm
- net N$13: track 0.00 -> 3.33 mm
- net MCLR: track 21.0 -> 18.6 mm
- net +5V: track 206.1 -> 204.1 mm
- net PGD: track 10.3 -> 11.9 mm
- net PGC: track 10.3 -> 11.9 mm
- net N$2: track 88.2 -> 89.5 mm
- net N$7: track 11.8 -> 11.2 mm
- net N$9: track 12.9 -> 12.2 mm
- net N$8: track 11.3 -> 10.6 mm
- net N$10: track 13.4 -> 12.7 mm
- net CLK: track 6.94 -> 7.58 mm
- net DIN: track 18.3 -> 18.8 mm
- net LOAD: track 14.7 -> 15.2 mm
Other:
- board text added: "Rev.B"
- board text removed: "Rev.A"
