File: DummyLoad.sch (EAGLE design)
At the start: 41 parts, among them IC1 LM324N, IC2 PIC18F2550_28DIP, IC3 MAX7219CNG, Q1 MTP3055, SW1 EC11B-V-T, X1 MINI-USB_B, X2 LOAD

Commit message: Update to latest local version
Parts:
- added C9: (no value), rcl:CPOL-EUD/7343-31R
- added R21: 10k, rcl:R-EU_R1206
Connections:
- new net N$13: IC3.ISET, R21.2
- net +5V: now also C9.+, R21.1
- net GND: now also C9.-
Changed lines of the file:
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@@
 <part name="GND20" library="supply1" deviceset="GND" device=""/>
 <part name="KK1" library="own-collection" deviceset="SK129-PAD" device="NO_RESTRICT" value="SK129-PADNO_RESTRICT"/>
+<part name="R21" library="rcl" deviceset="R-EU_" device="R1206" value="10k"/>
+<part name="P+10" library="supply1" deviceset="+5V" device=""/>
+<part name="C9" library="rcl" deviceset="CPOL-EU" device="D/7343-31R"/>
+<part name="GND21" library="supply1" deviceset="GND" device=""/>
 </parts>
 <sheets>
@@
 <instance part="X2" gate="-2" x="-177.8" y="63.5"/>
 <instance part="J1" gate="G$1" x="-175.26" y="96.52"/>
-<instance part="P+6" gate="1" x="-162.56" y="106.68"/>
+<instance part="P+6" gate="1" x="-160.02" y="106.68"/>
 <instance part="GND14" gate="1" x="-170.18" y="88.9"/>
 <instance part="C6" gate="G$1" x="-2.54" y="5.08"/>
@@
 <instance part="GND20" gate="1" x="-144.78" y="60.96"/>
 <instance part="KK1" gate="G$1" x="-139.7" y="66.04"/>
+<instance part="R21" gate="G$1" x="-2.54" y="27.94" rot="R270"/>
+<instance part="P+10" gate="1" x="-2.54" y="38.1"/>
+<instance part="C9" gate="G$1" x="-160.02" y="91.44"/>
+<instance part="GND21" gate="1" x="-160.02" y="81.28"/>
 </instances>
 <busses>
@@
 <pinref part="KK1" gate="G$1" pin="K@1"/>
 </segment>
+<segment>
+<pinref part="C9" gate="G$1" pin="-"/>
+<pinref part="GND21" gate="1" pin="GND"/>
+<wire x1="-160.02" y1="86.36" x2="-160.02" y2="83.82" width="0.1524" layer="91"/>
+</segment>
 </net>
 <net name="+5V" class="0">
@@
 <segment>
 <pinref part="P+6" gate="1" pin="+5V"/>
-<wire x1="-162.56" y1="99.06" x2="-162.56" y2="104.14" width="0.1524" layer="91"/>
+<wire x1="-160.02" y1="93.98" x2="-160.02" y2="99.06" width="0.1524" layer="91"/>
 <pinref part="D1" gate="G$1" pin="C"/>
+<pinref part="C9" gate="G$1" pin="+"/>
+<wire x1="-160.02" y1="99.06" x2="-160.02" y2="104.14" width="0.1524" layer="91"/>
+<wire x1="-162.56" y1="99.06" x2="-160.02" y2="99.06" width="0.1524" layer="91"/>
+<junction x="-160.02" y="99.06"/>
 </segment>
 <segment>
@@
 <wire x1="-27.94" y1="88.9" x2="-27.94" y2="86.36" width="0.1524" layer="91"/>
 <junction x="-27.94" y="86.36"/>
+</segment>
+<segment>
+<pinref part="R21" gate="G$1" pin="1"/>
+<pinref part="P+10" gate="1" pin="+5V"/>
+<wire x1="-2.54" y1="35.56" x2="-2.54" y2="33.02" width="0.1524" layer="91"/>
 </segment>
 </net>
@@
 </segment>
 </net>
+<net name="N$13" class="0">
+<segment>
+<pinref part="R21" gate="G$1" pin="2"/>
+<pinref part="IC3" gate="G$1" pin="ISET"/>
+<wire x1="-2.54" y1="22.86" x2="10.16" y2="22.86" width="0.1524" layer="91"/>
+</segment>
+</net>
